File: kicad/OceanNest_L/OceanNest_L.kicad_sch (KiCad schematic)
At the start: 34 parts, among them J1 TRRS_MJ-4PP-9, SW1 SW_Push, SW10 SW_Push, SW11 SW_Push, SW12 SW_Push, SW13 SW_Push, SW14 RotaryEncoder, SW2 SW_Push, SW3 SW_Push, SW4 SW_Push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

Commit message: feat: add new OceanNest_L and OceanNest_R PCB and project files for enhanced design capabilities
Parts:
- removed D13: D, kbd_Parts:Diode_SMD, symbol Device:D
- removed SW10: SW_Push, takashicompany:CherryMX_Hotswap_16m, symbol Switch:SW_Push
