File: kicad/OceanNest_L/OceanNest_L.kicad_sch (KiCad schematic)
At the start: 32 parts, among them J1 TRRS_MJ-4PP-9, SW1 SW_Push, SW11 SW_Push, SW12 SW_Push, SW13 SW_Push, SW14 RotaryEncoder, SW2 SW_Push, SW3 SW_Push, SW4 SW_Push, SW5 SW_Push, SW6 SW_Push, SW7 SW_Push, SW8 SW_Push, SW9 SW_Push, U1 XIAO-RP2040-DIP

Commit message: routing
Connections:
- net VCC: now also U1.1 (GPIO26/ADC0/A0); no longer U1.7 (GPIO0/TX)
- net data: now also U1.7 (GPIO0/TX); no longer U1.6 (GPIO7/SCL)
- net pin1: now also U1.2 (GPIO27/ADC1/A1); no longer U1.1 (GPIO26/ADC0/A0)
- net pin2: now also U1.3 (GPIO28/ADC2/A2); no longer U1.2 (GPIO27/ADC1/A1)
- net pin3: now also U1.4 (GPIO29/ADC3/A3); no longer U1.3 (GPIO28/ADC2/A2)
- net pin4: now also U1.5 (GPIO6/SDA); no longer U1.4 (GPIO29/ADC3/A3)
- net pin5: now also U1.6 (GPIO7/SCL); no longer U1.5 (GPIO6/SDA)
