File: kicad/OceanNest_L/OceanNest_L.kicad_pcb (KiCad board)
At the start: 2 copper layers, 113.5 x 88.7 mm, 36 parts, among them J1 TRRS_MJ-4PP-9, SW1 SW_Push, SW11 SW_Push, SW12 SW_Push, SW13 SW_Push, SW14 RotaryEncoder, SW2 SW_Push, SW3 SW_Push, SW4 SW_Push, SW5 SW_Push, SW6 SW_Push, SW7 SW_Push, SW8 SW_Push, SW9 SW_Push, U1 XIAO-RP2040-DIP

Commit message: routing
Parts:
- added hole2: Val**, kbd_Hole:m2_Spacer_Hole_hex, F.Cu at (173.0, 117.5)
- added hole2: Val**, kbd_Hole:m2_Spacer_Hole_hex, F.Cu at (100.5, 118.0)
- moved hole3 225.4 mm to (175.5, -57.0)
- moved hole4 225.4 mm to (175.5, -45.0)
- moved U1 143.7 mm to (182.5, 74.5), turned to 0 degrees
- moved hole1 90.0 mm to (163.0, 68.0)
- moved D17 73.9 mm to (186.0, 116.5)
- moved D12 72.3 mm to (182.5, 80.5)
- moved hole2 69.9 mm to (99.5, 70.0)
- moved D18 66.8 mm to (174.5, 110.5)
- moved SW5 63.0 mm to (111.8, 96.3)
- moved J1 62.7 mm to (188.8, 109.0)
- moved SW12 62.0 mm to (186.1, 134.9)
- moved SW13 62.0 mm to (203.0, 142.0)
- moved D8 60.5 mm to (130.0, 98.5)
- moved SW14 60.0 mm to (148.6, 119.0)
- moved D16 58.3 mm to (180.5, 122.5)
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Connections:
- U1 pad 1: pin1 -> VCC
- U1 pad 2: pin2 -> pin1
- U1 pad 3: pin3 -> pin2
- U1 pad 4: pin4 -> pin3
- U1 pad 5: pin5 -> pin4
- U1 pad 6: data -> pin5
- U1 pad 7: VCC -> data
Routing:
- net GND: track 90.6 -> 0.00 mm, vias 0 -> 65
- net pin2: track 59.1 -> 111.8 mm
- net VCC: track 108.4 -> 62.0 mm, vias 1 -> 0
- net pin5: track 104.3 -> 61.2 mm, vias 1 -> 2
- net data: track 79.9 -> 37.4 mm, vias 1 -> 2
- net REb: track 43.0 -> 72.8 mm
- net REa: track 42.7 -> 72.4 mm, vias 1 -> 0
- net pin1: track 118.6 -> 90.0 mm, vias 3 -> 2
- net Net-(D17-A): track 10.2 -> 37.0 mm
- net pin3: track 108.6 -> 90.9 mm
- net pin4: track 71.8 -> 88.6 mm, vias 1 -> 4
- net Net-(D6-A): track 12.3 -> 27.2 mm
- net Net-(D10-K): track 16.8 -> 30.7 mm, vias 0 -> 2
- net Net-(D18-K): track 96.1 -> 109.2 mm, vias 0 -> 4
- net Net-(D7-K): track 161.2 -> 172.9 mm, vias 3 -> 6
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- added copper zone on B.Cu, net GND
- added copper zone on F.Cu, net GND
Other:
- board size 113.5 x 88.7 mm -> 126.4 x 94.7 mm
