File: kicad/OceanNest_R/OceanNest_R.kicad_sch (KiCad schematic)
At the start: 38 parts, among them J21 TRRS_MJ-4PP-9, J22 Conn_01x07_Pin, SW21 SW_Push, SW22 SW_Push, SW23 SW_Push, SW24 SW_Push, SW25 SW_Push, SW26 SW_Push, SW27 SW_Push, SW28 SW_Push, SW29 SW_Push, SW30 SW_Push, SW31 SW_Push, SW32 SW_Push, SW33 SW_Push, SW34 SW_Push, SW35 SW_Push, U22 XIAO-RP2040-DIP

Commit message: feat: add new OceanNest_L and OceanNest_R PCB and project files for enhanced design capabilities
Parts:
- removed D37: D, kbd_Parts:Diode_SMD, symbol Device:D
- removed SW33: SW_Push, takashicompany:CherryMX_Hotswap_16m, symbol Switch:SW_Push
- renumbered D38 to D37, D39 to D38, D40 to D39, SW34 to SW33, SW35 to SW34, U22 to U21
