File: kicad/OceanNest_R/OceanNest_R.kicad_sch (KiCad schematic)
At the start: 36 parts, among them J21 TRRS_MJ-4PP-9, J22 Conn_01x07_Pin, SW21 SW_Push, SW22 SW_Push, SW23 SW_Push, SW24 SW_Push, SW25 SW_Push, SW26 SW_Push, SW27 SW_Push, SW28 SW_Push, SW29 SW_Push, SW30 SW_Push, SW31 SW_Push, SW32 SW_Push, SW33 SW_Push, SW34 SW_Push, U21 XIAO-RP2040-DIP

Commit message: routing
Connections:
- net GND: now also U21.1 (GPIO26/ADC0/A0); no longer U21.7 (GPIO0/TX)
- net data: now also U21.7 (GPIO0/TX); no longer U21.6 (GPIO7/SCL)
- net pin1: now also U21.2 (GPIO27/ADC1/A1); no longer U21.1 (GPIO26/ADC0/A0)
- net pin2: now also U21.3 (GPIO28/ADC2/A2); no longer U21.2 (GPIO27/ADC1/A1)
- net pin3: now also U21.4 (GPIO29/ADC3/A3); no longer U21.3 (GPIO28/ADC2/A2)
- net pin4: now also U21.5 (GPIO6/SDA); no longer U21.4 (GPIO29/ADC3/A3)
- net pin5: now also U21.6 (GPIO7/SCL); no longer U21.5 (GPIO6/SDA)
